File: hardware/relay/knuth-gateway.kicad_pcb (KiCad board)
At the start: 2 copper layers, 65.4 x 57.1 mm, 12 parts, among them J1 Screw_Terminal_01x03, J2 Screw_Terminal_01x03, J3 FeatherLora1, J4 FeatherLora2, J5 Conn_01x07_Female, SW2 SW_SPDT

Commit message: update
Parts:
- added RA1: R, Resistor_THT:R_Axial_DIN0207_L6.3mm_D2.5mm_P2.54mm_Vertical, F.Cu at (54.6, 19.1)
- added SW1: SW_SPDT, Connector_PinSocket_2.54mm:PinSocket_1x03_P2.54mm_Vertical, F.Cu at (62.9, 33.0)
- moved J2 4.58 mm to (64.8, 27.3)
- moved J1 2.84 mm to (64.8, 12.7)
- moved BT1 1.91 mm to (62.2, 47.6)
- moved SW2 0.64 mm to (60.3, 55.2)
- renumbered D1 to D13, RO1 to R1, R1 to R13
Connections:
- J4 pad 7: (no net) -> A2
Routing:
- net A2: track 0.00 -> 25.1 mm
- net Net-(RA1-Pad2): track 0.00 -> 17.5 mm, vias 0 -> 2
- net GND: track 138.5 -> 151.8 mm
- net +3V3: track 119.5 -> 128.4 mm
- net Net-(BT1-Pad1): track 10.6 -> 8.94 mm
- net D10: track 83.3 -> 81.7 mm, vias 2 -> 0
- net VBAT: track 45.9 -> 47.0 mm
- net D12: track 9.94 -> 9.20 mm
Other:
- board size 65.4 x 57.1 mm -> 65.4 x 58.4 mm

Commit message: update
Parts:
- moved SW2 4.26 mm to (62.2, 51.4)
- moved BT1 3.18 mm to (64.8, 45.7)
Routing:
- net GND: track 151.8 -> 148.9 mm
- net A2: track 25.1 -> 22.8 mm
- net Net-(BT1-Pad1): track 8.94 -> 6.77 mm

Commit message: shrortened jumper wires
Routing:
- net GND: track 148.9 -> 155.6 mm
- net +3V3: track 128.4 -> 132.1 mm
Changed lines of the file:
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@@
     (thickness 1.6)
     (drawings 10)
-    (tracks 133)
+    (tracks 139)
     (zones 0)
     (modules 14)
@@
     (uvia_drill 0.1)
     (add_net +3V3)
-    (add_net A0)
-    (add_net A1)
     (add_net A2)
-    (add_net A3)
-    (add_net A4)
-    (add_net AREF)
-    (add_net D0)
-    (add_net D1)
     (add_net D10)
-    (add_net D11)
     (add_net D12)
-    (add_net D13)
-    (add_net D5)
     (add_net D6)
-    (add_net D9)
-    (add_net EN)
     (add_net GND)
-    (add_net MISO)
-    (add_net MOSI)
     (add_net "Net-(BT1-Pad1)")
     (add_net "Net-(D13-Pad2)")
-    (add_net "Net-(J5-Pad2)")
-    (add_net "Net-(J5-Pad5)")
-    (add_net "Net-(J5-Pad7)")
     (add_net "Net-(RA1-Pad2)")
-    (add_net "Net-(SW2-Pad1)")
-    (add_net RESET)
-    (add_net SCK)
     (add_net SCL)
     (add_net SDA)
     (add_net VBAT)
-    (add_net VBUS)
   )
   (module Connector_PinSocket_2.54mm:PinSocket_1x03_P2.54mm_Vertical (layer F.Cu)
@@
   (gr_line (start 67.31 1.27) (end 9.525 1.27) (layer Edge.Cuts) (width 0.15))
   (segment (start 49.6062 28.0162) (end 49.53 27.94) (width 1.905) (layer B.Cu) (net 0) (status 30))
-  (via (at 12.7 33.02) (size 1.778) (drill 0.889) (layers F.Cu B.Cu) (net 1))
-  (segment (start 15.24 35.56) (end 12.7 33.02) (width 1.7) (layer F.Cu) (net 1))
+  (via (at 12.7 41.91) (size 1.778) (drill 0.889) (layers F.Cu B.Cu) (net 1))
   (segment (start 12.7 21.59) (end 12.7 33.02) (width 1.7) (layer B.Cu) (net 1))
   (segment (start 21.59 16.51) (end 17.78 16.51) (width 1.7) (layer B.Cu) (net 1))
@@
   (via (at 19.685 41.91) (size 1.778) (drill 0.889) (layers F.Cu B.Cu) (net 1))
   (segment (start 21.59 40.005) (end 19.685 41.91) (width 1.7) (layer B.Cu) (net 1))
-  (segment (start 15.24 37.465) (end 15.24 35.56) (width 1.7) (layer F.Cu) (net 1))
-  (segment (start 19.685 41.91) (end 15.24 37.465) (width 1.7) (layer F.Cu) (net 1))
   (segment (start 66.467056 9.2) (end 67.31 10.042944) (width 1.7) (layer B.Cu) (net 1))
   (segment (start 64.77 9.2) (end 66.467056 9.2) (width 1.7) (layer B.Cu) (net 1))
@@
   (segment (start 46.355 43.18) (end 49.53 43.18) (width 1.7) (layer B.Cu) (net 1))
   (segment (start 31.75 48.26) (end 34.29 45.72) (width 1.7) (layer F.Cu) (net 1))
-  (via (at 25.4 48.26) (size 1.778) (drill 0.889) (layers F.Cu B.Cu) (net 1))
+  (via (at 28.575 51.435) (size 1.778) (drill 0.889) (layers F.Cu B.Cu) (net 1))
   (segment (start 19.685 41.91) (end 19.685 42.545) (width 1.7) (layer B.Cu) (net 1))
   (segment (start 19.685 42.545) (end 25.4 48.26) (width 1.7) (layer B.Cu) (net 1))
-  (segment (start 25.4 48.26) (end 30.48 48.26) (width 1.7) (layer F.Cu) (net 1))
-  (segment (start 30.48 48.26) (end 31.75 48.26) (width 1.7) (layer F.Cu) (net 1))
   (via (at 34.29 45.72) (size 1.778) (drill 0.889) (layers F.Cu B.Cu) (net 1))
   (segment (start 46.355 43.18) (end 41.275 38.1) (width 1.7) (layer B.Cu) (net 1))
   (segment (start 36.83 38.1) (end 41.275 38.1) (width 1.7) (layer B.Cu) (net 1))
+  (segment (start 12.7 33.02) (end 12.7 41.91) (width 1.7) (layer B.Cu) (net 1))
+  (segment (start 19.685 41.91) (end 12.7 41.91) (width 1.7) (layer F.Cu) (net 1))
+  (segment (start 25.4 48.26) (end 26.035 48.895) (width 1.7) (layer B.Cu) (net 1))
+  (segment (start 26.035 48.895) (end 26.67 49.53) (width 1.7) (layer B.Cu) (net 1))
+  (segment (start 26.67 49.53) (end 27.305 50.165) (width 1.7) (layer B.Cu) (net 1))
+  (segment (start 27.305 50.165) (end 27.94 50.8) (width 1.7) (layer B.Cu) (net 1))
+  (segment (start 31.75 48.26) (end 28.575 51.435) (width 1.7) (layer F.Cu) (net 1))
+  (segment (start 27.94 50.8) (end 28.575 51.435) (width 1.7) (layer B.Cu) (net 1))
   (segment (start 55.245 5.715) (end 55.245 8.89) (width 1.7) (layer B.Cu) (net 2))
   (segment (start 64.12 5.7) (end 64.135 5.715) (width 1.905) (layer B.Cu) (net 2))
@@
   (segment (start 29.21 12.7) (end 25.4 8.89) (width 1.7) (layer B.Cu) (net 8))
   (segment (start 25.4 8.89) (end 21.59 8.89) (width 1.7) (layer B.Cu) (net 8))
-  (segment (start 30.48 52.07) (end 24.13 52.07) (width 1.7) (layer B.Cu) (net 9))
   (segment (start 44.45 48.26) (end 40.64 52.07) (width 1.7) (layer B.Cu) (net 9))
   (segment (start 49.53 48.26) (end 44.45 48.26) (width 1.7) (layer B.Cu) (net 9))
-  (via (at 30.48 52.07) (size 1.778) (drill 0.889) (layers F.Cu B.Cu) (net 9))
-  (via (at 40.64 52.07) (size 1.778) (drill 0.889) (layers F.Cu B.Cu) (net 9))
-  (segment (start 40.64 52.07) (end 30.48 52.07) (width 1.7) (layer F.Cu) (net 9))
-  (segment (start 19.04 21.59) (end 16.51 24.12) (width 1.7) (layer B.Cu) (net 9))
-  (segment (start 21.59 21.59) (end 19.04 21.59) (width 1.7) (layer B.Cu) (net 9))
-  (segment (start 16.51 44.45) (end 17.78 45.72) (width 1.7) (layer B.Cu) (net 9))
-  (segment (start 16.51 24.12) (end 16.51 44.45) (width 1.7) (layer B.Cu) (net 9))
-  (segment (start 24.13 52.07) (end 17.78 45.72) (width 1.7) (layer B.Cu) (net 9))
+  (via (at 33.655 54.61) (size 1.778) (drill 0.889) (layers F.Cu B.Cu) (net 9))
   (segment (start 64.77 12.7) (end 61.87 12.7) (width 1.7) (layer B.Cu) (net 9))
   (segment (start 64.77 27.305) (end 53.975 27.305) (width 1.7) (layer B.Cu) (net 9))
@@
   (segment (start 60.6 11.43) (end 61.87 12.7) (width 1.7) (layer B.Cu) (net 9))
   (segment (start 55.245 11.43) (end 60.6 11.43) (width 1.7) (layer B.Cu) (net 9))
+  (segment (start 40.005 51.435) (end 40.64 52.07) (width 1.7) (layer B.Cu) (net 9))
+  (segment (start 38.735 50.165) (end 38.735 50.165) (width 1.7) (layer B.Cu) (net 9))
+  (segment (start 19.04 21.59) (end 21.59 21.59) (width 1.7) (layer B.Cu) (net 9))
+  (segment (start 16.51 44.45) (end 16.51 24.12) (width 1.7) (layer B.Cu) (net 9))
+  (segment (start 33.655 54.61) (end 26.67 54.61) (width 1.7) (layer B.Cu) (net 9))
+  (segment (start 16.51 24.12) (end 19.04 21.59) (width 1.7) (layer B.Cu) (net 9))
+  (segment (start 26.67 54.61) (end 16.51 44.45) (width 1.7) (layer B.Cu) (net 9))
+  (segment (start 38.735 50.165) (end 40.005 51.435) (width 1.7) (layer B.Cu) (net 9))
+  (via (at 38.735 50.165) (size 1.778) (drill 0.889) (layers F.Cu B.Cu) (net 9))
+  (segment (start 38.1 50.165) (end 33.655 54.61) (width 1.7) (layer F.Cu) (net 9))
+  (segment (start 38.735 50.165) (end 38.1 50.165) (width 1.7) (layer F.Cu) (net 9))
   (segment (start 21.59 29.21) (end 21.59 34.925) (width 1.7) (layer B.Cu) (net 10))
   (segment (start 51.435 35.56) (end 49.53 35.56) (width 1.7) (layer B.Cu) (net 11))
